File: test.kicad_pcb (KiCad board)
At the start: 2 copper layers, 44.4 x 26.5 mm, 2 parts

Commit message: upadet pcb
Parts:
- moved R1 3.78 mm to (140.2, 80.5)
Routing:
- net Net-(R1-Pad2): track 4.21 -> 8.27 mm
- net Net-(R1-Pad1): track 4.21 -> 8.27 mm
Changed lines of the file:
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@@
 	(footprint "Resistor_SMD:R_1210_3225Metric_Pad1.30x2.65mm_HandSolder"
 		(layer "F.Cu")
-		(at 143.48 82.355)
+		(at 140.2 80.48)
 		(descr "Resistor SMD 1210 (3225 Metric), square (rectangular) end terminal, IPC-7351 nominal with elongated pad for handsoldering. (Body size source: IPC-SM-782 page 72, https://www.pcb-3d.com/wordpress/wp-content/uploads/ipc-sm-782a_amendment_1_and_2.pdf), generated with kicad-footprint-generator")
 		(tags "resistor handsolder")
@@
 	)
 	(segment
+		(start 141.75 80.48)
+		(end 143.625 82.355)
+		(width 0.2)
+		(layer "F.Cu")
+		(net 1)
+	)
+	(segment
+		(start 143.625 82.355)
+		(end 145.03 82.355)
+		(width 0.2)
+		(layer "F.Cu")
+		(net 1)
+	)
+	(segment
 		(start 141.93 82.355)
 		(end 141.93 86.565)
 		(width 0.2)
 		(layer "F.Cu")
+		(net 2)
+	)
+	(segment
+		(start 140.525 82.355)
+		(end 141.93 82.355)
+		(width 0.2)
+		(layer "F.Cu")
+		(net 2)
+	)
+	(segment
+		(start 138.65 80.48)
+		(end 140.525 82.355)
+		(width 0.2)
+		(layer "F.Cu")

Commit message: update pcb
Routing:
- net Net-(R1-Pad2): track 8.27 -> 9.15 mm
Changed lines of the file:
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@@
 	)
 	(segment
-		(start 145.03 82.355)
+		(start 144.69 80.51)
+		(end 145.03 80.85)
+		(width 0.2)
+		(layer "F.Cu")
+		(net 1)
+	)
+	(segment
+		(start 141.75 80.48)
+		(end 141.78 80.51)
+		(width 0.2)
+		(layer "F.Cu")
+		(net 1)
+	)
+	(segment
+		(start 145.03 80.85)
 		(end 145.03 86.565)
 		(width 0.2)
@@
 	)
 	(segment
-		(start 141.75 80.48)
-		(end 143.625 82.355)
+		(start 141.78 80.51)
+		(end 144.69 80.51)
 		(width 0.2)
 		(layer "F.Cu")
-		(net 1)
-	)
-	(segment
-		(start 143.625 82.355)
-		(end 145.03 82.355)
-		(width 0.2)
-		(layer "F.Cu")

Commit message: update pcb
Routing:
- net Net-(R1-Pad1): track 8.27 -> 11.4 mm
Changed lines of the file:
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@@
 	)
 	(segment
-		(start 141.93 82.355)
+		(start 137.72 82.355)
 		(end 141.93 86.565)
-		(width 0.2)
-		(layer "F.Cu")
-		(net 2)
-	)
-	(segment
-		(start 140.525 82.355)
-		(end 141.93 82.355)
 		(width 0.2)
 		(layer "F.Cu")
@@
 		(width 0.2)
 		(layer "F.Cu")
+		(net 2)
+	)
+	(segment
+		(start 140.525 82.355)
+		(end 137.72 82.355)
+		(width 0.2)
+		(layer "F.Cu")

Commit message: update pcb
Routing:
- net Net-(R1-Pad2): track 9.15 -> 10.9 mm
Changed lines of the file:
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@@
 		(tags "resistor handsolder")
 		(property "Reference" "R2"
-			(at 4.15 -1.865 0)
+			(at 4.15 -0.275 0)
 			(layer "F.SilkS")
 			(effects
@@
 	)
 	(segment
-		(start 144.69 80.51)
-		(end 145.03 80.85)
+		(start 141.78 80.51)
+		(end 144.69 80.51)
 		(width 0.2)
 		(layer "F.Cu")
@@
 	)
 	(segment
-		(start 145.03 80.85)
+		(start 144.69 80.51)
+		(end 147.15 82.97)
+		(width 0.2)
+		(layer "F.Cu")
+		(net 1)
+	)
+	(segment
+		(start 147.15 82.97)
+		(end 147.15 84.445)
+		(width 0.2)
+		(layer "F.Cu")
+		(net 1)
+	)
+	(segment
+		(start 147.15 84.445)
 		(end 145.03 86.565)
 		(width 0.2)
 		(layer "F.Cu")
-		(net 1)
-	)
-	(segment
-		(start 141.78 80.51)
-		(end 144.69 80.51)
-		(width 0.2)
-		(layer "F.Cu")

Commit message: update pcb
Routing:
- net Net-(R1-Pad2): track 10.9 -> 12.3 mm
Changed lines of the file:
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@@
 	(segment
 		(start 141.78 80.51)
-		(end 144.69 80.51)
+		(end 147.15 80.51)
 		(width 0.2)
 		(layer "F.Cu")
@@
 	)
 	(segment
-		(start 144.69 80.51)
-		(end 147.15 82.97)
+		(start 147.15 84.445)
+		(end 145.03 86.565)
 		(width 0.2)
 		(layer "F.Cu")
@@
 	)
 	(segment
-		(start 147.15 82.97)
+		(start 147.15 80.51)
 		(end 147.15 84.445)
 		(width 0.2)
 		(layer "F.Cu")
-		(net 1)
-	)
-	(segment
-		(start 147.15 84.445)
-		(end 145.03 86.565)
-		(width 0.2)
-		(layer "F.Cu")

Commit message: update pcb
Routing:
- net Net-(R1-Pad1): track 11.4 -> 23.8 mm
Changed lines of the file:
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@@
 	)
 	(segment
-		(start 137.72 82.355)
+		(start 131.535 82.355)
+		(end 135.745 86.565)
+		(width 0.2)
+		(layer "F.Cu")
+		(net 2)
+	)
+	(segment
+		(start 135.745 86.565)
 		(end 141.93 86.565)
 		(width 0.2)
@@
 	(segment
 		(start 140.525 82.355)
-		(end 137.72 82.355)
+		(end 131.535 82.355)
 		(width 0.2)
 		(layer "F.Cu")

Commit message: update pcb
Routing:
- net Net-(R1-Pad2): track 12.3 -> 17.9 mm
Changed lines of the file:
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@@
+	)
+	(segment
+		(start 151.085 80.51)
+		(end 145.03 86.565)
+		(width 0.2)
+		(layer "F.Cu")
+		(net 1)
 	)
 	(segment
 		(start 141.78 80.51)
-		(end 147.15 80.51)
+		(end 151.085 80.51)
 		(width 0.2)
 		(layer "F.Cu")
@@
 		(width 0.2)
 		(layer "F.Cu")
-		(net 1)
-	)
-	(segment
-		(start 147.15 84.445)
-		(end 145.03 86.565)
-		(width 0.2)
-		(layer "F.Cu")
-		(net 1)
-	)
-	(segment
-		(start 147.15 80.51)
-		(end 147.15 84.445)
-		(width 0.2)
-		(layer "F.Cu")

Commit message: update pcb
Routing:
- net Net-(R1-Pad1): track 23.8 -> 25.6 mm
Changed lines of the file:
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@@
-	)
-	(segment
-		(start 131.535 82.355)
-		(end 135.745 86.565)
-		(width 0.2)
-		(layer "F.Cu")
-		(net 2)
-	)
-	(segment
-		(start 135.745 86.565)
-		(end 141.93 86.565)
-		(width 0.2)
-		(layer "F.Cu")
-		(net 2)
 	)
 	(segment
@@
 		(width 0.2)
 		(layer "F.Cu")
+		(net 2)
+	)
+	(segment
+		(start 131.535 82.355)
+		(end 137.96 88.78)
+		(width 0.2)
+		(layer "F.Cu")
+		(net 2)
+	)
+	(segment
+		(start 137.96 88.78)
+		(end 139.715 88.78)
+		(width 0.2)
+		(layer "F.Cu")
+		(net 2)
+	)
+	(segment
+		(start 139.715 88.78)
+		(end 141.93 86.565)
+		(width 0.2)
+		(layer "F.Cu")
